File: ESP32Driver.brd (EAGLE design)
At the start: 59.7 x 36.5 mm, 90 parts, among them IC1 ESP-WROOM-32_VIA, IC3 FT231XQ, SW2 434111025826, T1.1 BC847A, T1.2 BC847A, T1.3 BC847A, T1.4 BC847A, X1 USB

Commit message: delete GPIO2 pullup resistor
Parts:
- removed R1.16: 10k, rcl:R0805
Connections:
- net +3V3: no longer R1.16.1
- net GPIO2: no longer R1.16.2
Routing:
- net GPIO2: track 23.9 -> 21.0 mm
- net +3V3: track 46.4 -> 44.0 mm
- net GPIO18: track 37.9 -> 37.0 mm
Changed lines of the file:
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@@
 <?xml version="1.0" encoding="utf-8"?>
 <!DOCTYPE eagle SYSTEM "eagle.dtd">
-<eagle version="9.4.0">
+<eagle version="9.6.2">
 <drawing>
 <settings>
@@
 </layers>
 <board>
-<fusionsync huburn="a.cGVyc29uYWw6dWUyZDczNzY0" projecturn="a.cGVyc29uYWw6dWUyZDczNzY0IzIwMTgxMDEwMTUzNzI5MTc2" f3durn="urn:adsk.wipprod:dm.lineage:rg9JTajcTwaWEXiMoO7pRw" pcbguid="91c40198-4244-4f42-9bba-0616e2d85463" lastpulledtime="" lastsyncedchangeguid="decd244c-18bb-9ce4-2c37-a45b05c47c5b"/>
+<fusionsync huburn="a.cGVyc29uYWw6dWUyZDczNzY0" projecturn="a.cGVyc29uYWw6dWUyZDczNzY0IzIwMTgxMDEwMTUzNzI5MTc2" f3durn="urn:adsk.wipprod:dm.lineage:rg9JTajcTwaWEXiMoO7pRw" pcbguid="91c40198-4244-4f42-9bba-0616e2d85463" lastpulledtime="" lastsyncedchangeguid="decd244c-18bb-9ce4-2c37-a45b05c47c5b" latestrevisionid="" lastsyncedrevisionid="" lastboardhashguid="" lastpushedtime="" linktopcb3d="false"/>
 <plain>
 <wire x1="-0.127" y1="0" x2="59.543" y2="0" width="0" layer="20"/>
@@
 <attribute name="VALUE" x="49.53" y="23.876" size="1.27" layer="28" rot="MR180"/>
 </element>
-<element name="R1.16" library="rcl" package="R0805" value="10k" x="22.225" y="19.812" smashed="yes">
-<attribute name="NAME" x="20.066" y="17.78" size="1.016" layer="25" font="vector"/>
-<attribute name="VALUE" x="19.177" y="16.383" size="1.016" layer="27" font="vector"/>
-</element>
 <element name="R1.2" library="rcl" package="R0805" value="10k" x="47.625" y="11.938" smashed="yes" rot="MR0">
 <attribute name="NAME" x="48.26" y="13.208" size="1.27" layer="26" rot="MR0"/>
@@
 <contactref element="C1.3" pad="+"/>
 <contactref element="C1.8" pad="1"/>
-<contactref element="R1.16" pad="1"/>
 <contactref element="R1.1" pad="1"/>
 <contactref element="R1.2" pad="1"/>
@@
 <wire x1="22.7496" y1="23.2576" x2="23.114" y2="23.622" width="0.1524" layer="16"/>
 <wire x1="21.5354" y1="23.0594" x2="22.6156875" y2="23.0594" width="0.1524" layer="16"/>
-<wire x1="21.275" y1="19.812" x2="23.114" y2="21.651" width="0.1524" layer="1"/>
-<wire x1="23.114" y1="21.651" x2="23.114" y2="23.622" width="0.1524" layer="1"/>
 <wire x1="24.021" y1="18.939" x2="24.749" y2="18.939" width="0.1524" layer="16"/>
 <wire x1="24.749" y1="18.939" x2="25.146" y2="18.542" width="0.1524" layer="16"/>
@@
 <wire x1="25.146" y1="18.542" x2="25.146" y2="15.0142" width="0.1524" layer="1"/>
 <wire x1="25.146" y1="15.0142" x2="25.019" y2="14.8872" width="0.1524" layer="1"/>
-<wire x1="21.275" y1="19.812" x2="22.545" y2="18.542" width="0.1524" layer="1"/>
-<wire x1="22.545" y1="18.542" x2="25.146" y2="18.542" width="0.1524" layer="1"/>
 <via x="50.038" y="13.335" extent="1-16" drill="0.35"/>
 <wire x1="50.038" y1="13.335" x2="51.181" y2="14.478" width="0.254" layer="1"/>
@@
 <via x="10.033" y="13.081" extent="1-16" drill="0.35"/>
 <wire x1="5.842" y1="13.081" x2="10.033" y2="13.081" width="0.508" layer="1"/>
+<wire x1="23.114" y1="19.431" x2="24.003" y2="18.542" width="0.1524" layer="1"/>
+<wire x1="24.003" y1="18.542" x2="25.146" y2="18.542" width="0.1524" layer="1"/>
+<wire x1="23.114" y1="23.622" x2="23.114" y2="19.431" width="0.1524" layer="1"/>
 </signal>
 <signal name="MC_RX">
@@
 <signal name="GPIO2">
 <contactref element="IC1" pad="24"/>
-<contactref element="R1.16" pad="2"/>
 <contactref element="T1.2" pad="3"/>
 <contactref element="T1.1" pad="3"/>
@@
 <wire x1="37.592" y1="11.176" x2="37.734" y2="11.034" width="0.1524" layer="1"/>
 <wire x1="37.734" y1="11.034" x2="39.932" y2="11.034" width="0.1524" layer="1"/>
-<wire x1="23.175" y1="19.812" x2="25.992" y2="19.812" width="0.1524" layer="1"/>
-<wire x1="25.992" y1="19.812" x2="26.035" y2="19.855" width="0.1524" layer="1"/>
 </signal>
 <signal name="U2RXD">
@@
 <via x="47.117" y="5.9916" extent="1-16" drill="0.35"/>
 <wire x1="47.117" y1="5.9916" x2="38.081325" y2="5.9916" width="0.1524" layer="16"/>
-<wire x1="17.526" y1="13.335" x2="18.161" y2="12.7" width="0.1524" layer="1"/>
 <wire x1="17.526" y1="13.335" x2="18.288" y2="12.573" width="0.1524" layer="1"/>
 <wire x1="18.288" y1="12.573" x2="18.288" y2="8.509" width="0.1524" layer="1"/>
@@
 <wire x1="17.526" y1="28.575" x2="15.7932" y2="26.8422" width="0.508" layer="16"/>
 <wire x1="15.7932" y1="26.8422" x2="13.12723125" y2="26.8422" width="0.508" layer="16"/>
-<wire x1="8.951" y1="9.017" x2="8.951" y2="8.89" width="0.508" layer="16"/>
-<wire x1="9.017" y1="9.017" x2="8.951" y2="9.017" width="0.508" layer="16"/>
 <wire x1="19.624" y1="34.29" x2="15.748" y2="34.29" width="0.508" layer="16"/>
 <wire x1="15.748" y1="34.29" x2="15.494" y2="34.544" width="0.508" layer="16"/>
-<wire x1="8.951" y1="8.89" x2="9.652" y2="8.89" width="0.508" layer="16"/>
-<wire x1="9.652" y1="8.89" x2="10.315" y2="8.227" width="0.508" layer="16"/>
-<wire x1="10.315" y1="8.227" x2="10.315" y2="7.84565625" width="0.508" layer="16"/>
+<wire x1="10.315" y1="7.84565625" x2="10.315" y2="8.227" width="0.508" layer="16"/>
 <wire x1="10.315" y1="7.84565625" x2="10.823" y2="7.33765625" width="0.508" layer="16"/>
 <wire x1="10.823" y1="5.461" x2="11.27" y2="5.014" width="0.508" layer="16"/>
@@
 <wire x1="1.062" y1="31.369" x2="2.54" y2="31.369" width="0.508" layer="16"/>
 <wire x1="0.427" y1="30.734" x2="0.427" y2="20.782" width="0.508" layer="16"/>
-<wire x1="3.6357" y1="20.066" x2="3.6967" y2="20.127" width="0.508" layer="16"/>
 <wire x1="1.905" y1="20.127" x2="3.6967" y2="20.127" width="0.508" layer="16"/>
 <wire x1="0.427" y1="20.782" x2="1.082" y2="20.127" width="0.508" layer="16"/>
@@
 <wire x1="12.5056" y1="17.45825625" x2="12.18134375" y2="17.134" width="0.508" layer="16"/>
 <wire x1="10.122" y1="16.726" x2="10.122" y2="16.04944375" width="0.508" layer="16"/>
-<wire x1="8.951" y1="14.87844375" x2="8.951" y2="8.89" width="0.508" layer="16"/>
-<wire x1="10.122" y1="16.04944375" x2="8.951" y2="14.87844375" width="0.508" layer="16"/>
+<wire x1="10.122" y1="16.04944375" x2="9.101278125" y2="15.028721875" width="0.508" layer="16"/>
 <wire x1="12.5056" y1="26.22056875" x2="12.5056" y2="17.45825625" width="0.508" layer="16"/>
 <wire x1="10.53" y1="17.134" x2="10.122" y2="16.726" width="0.508" layer="16"/>
+<wire x1="9.101278125" y1="15.028721875" x2="9.101278125" y2="9.040278125" width="0.508" layer="16"/>
+<wire x1="9.101278125" y1="9.040278125" x2="8.951" y2="8.89" width="0.508" layer="16"/>
+<wire x1="10.315" y1="8.227" x2="9.501721875" y2="9.040278125" width="0.508" layer="16"/>
+<wire x1="9.501721875" y1="9.040278125" x2="9.101278125" y2="9.040278125" width="0.508" layer="16"/>
 </signal>
 <signal name="+5V">
